Commit message: gazebo plugin tested with the vi-sensor- looks good.

File: resources/models/gimbal_snippets.xacro (robot description, xacro)
@@ -2,10 +2,10 @@
 <robot xmlns:xacro="http://www.ros.org/wiki/xacro">
     <xacro:macro name="gimbal_base_joint" params="link_name joint_name child_link visible rpy parent_link *origin">
-        <joint name="gimbal_fix" type="fixed">
+         <joint name="gimbal_fix" type="prismatic"> <!-- prismatic joint with zero limits(default) is a hack for a fixed joint (needed on gazebo7)-->
             <parent link="${parent_link}"/>
             <child link="${link_name}"/>
             <axis xyz="1 0 0"/>
             <dynamics damping="0"/>
-            <dynamics friction="0"/>
+            <dynamics friction="100"/>
             <limit velocity="1e+16" effort="1e+16" />
             <xacro:insert_block name="origin" />
@@ -31,5 +31,5 @@
             <axis xyz="1 0 0"/>
             <dynamics damping="0"/>
-            <dynamics friction="0"/>
+            <dynamics friction="1000"/>
             <limit velocity="1e+16" effort="1e+16" />
             <origin xyz="0 0 0" rpy="${rpy}"/>
@@ -107,9 +107,9 @@
     </xacro:macro>
     <xacro:macro name="bottom_1D_gimbal" params="namespace parent_link *origin visible">
-        <gimbal_base_joint  joint_name="pitch_joint" link_name="gimbal_base_link" child_link="camera_mount_link" visible="${visible}" rpy="0 0 ${pi/2}" parent_link="${parent_link}">
+        <gimbal_base_joint  joint_name="${namespace}/pitch_joint" link_name="${namespace}/gimbal_base_link" child_link="${namespace}/camera_mount_link" visible="${visible}" rpy="0 0 ${pi/2}" parent_link="${parent_link}">
             <xacro:insert_block name="origin" />
         </gimbal_base_joint>
-        <link name='camera_mount_link'>
- <xacro:if value="${visible}">
+        <link name='${namespace}/camera_mount_link'>
+          <xacro:if value="${visible}">
             <visual >
                 <origin xyz="0 0 0"/>
@@ -118,9 +118,9 @@
                 </geometry>
             </visual>
- </xacro:if>
+           </xacro:if>
             <inertial>
                 <mass value="1e-5" />
-        <origin xyz="0 0 0" rpy="0 0 0" />
-        <inertia ixx="1e-6" ixy="0" ixz="0" iyy="1e-6" iyz="0" izz="1e-6" />
+		<origin xyz="0 0 0" rpy="0 0 0" />
+		<inertia ixx="1e-6" ixy="0" ixz="0" iyy="1e-6" iyz="0" izz="1e-6" />
             </inertial>
         </link>
@@ -128,10 +128,10 @@
             <plugin name="gimbal_controller" filename="libgazebo_poltergeist_gimbal_plugin.so">
                 <robot_namespace>/${namespace}</robot_namespace>
-                <pitch_joint_name>pitch_joint</pitch_joint_name>
+                <pitch_joint_name>${namespace}/pitch_joint</pitch_joint_name>
                 <pitch_direction>1</pitch_direction>
                 <pitch_zero>0</pitch_zero>
-                <gimbal_angular_velocity>0.3</gimbal_angular_velocity>
+                <gimbal_angular_velocity>0.5</gimbal_angular_velocity>
                 <ref_base_link>${parent_link}</ref_base_link>
-                <camera_link>camera_mount_link</camera_link>
+                <camera_link>${namespace}/camera_mount_link</camera_link>
             </plugin>
         </gazebo>
